File: KiCAD files/reflow.sch (KiCad schematic (older format))
At the start: 51 parts, among them J1 Screw_Terminal_01x02, J2 Screw_Terminal_01x02, J3 Conn_01x06_Female, J4 Conn_01x06_Female, J5 Conn_01x06_Female, J6 Screw_Terminal_01x02, J7 Screw_Terminal_01x02, U1 MOC3063M, U2 HLK-PM03, U3 ESP-12E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

Commit message: deleted outdated gerbers
Parts:
- U1: symbol Relay_SolidState:MOC3063M -> reflow-rescue:MOC3063M-Relay_SolidState
Changed lines of the file:
@@
 EESchema Schematic File Version 4
-LIBS:reflow-cache
-EELAYER 26 0
+EELAYER 30 0
 EELAYER END
 $Descr A4 11693 8268
@@
 $EndDescr
 $Comp
-L Relay_SolidState:MOC3063M U1
+L reflow-rescue:MOC3063M-Relay_SolidState U1
 U 1 1 5BEB127F
 P 2550 6750
